File: RSC-LV3-SwitchSense.kicad_pcb (KiCad board)
At the start: 2 copper layers, 140 x 85 mm, 183 parts, among them J1 FTSH-105-01-L-DV-K-A, J10 Molex 43045-0400, J11 Molex 43045-0400, J12 Molex 43045-0400, J13 Molex 43045-0400, J14 Molex 43045-0400, J15 Molex 43045-0400, J16 Molex 43650-0200, J2 USB_C_Receptacle_USB2.0_16P, J3 Molex 43650-0500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

Commit message: r0 final
Parts:
- removed D4, D9: D_Zener, Diode_SMD:D_SOD-323_HandSoldering
Routing:
- net V_SENSE_12: track 67.8 -> 65.6 mm
- net V_SENSE_5: track 37.7 -> 35.6 mm
